Commit message: weird collision in pybullet, going to test in gazebo

File: tmm_description/robot.urdf (robot description, URDF)
Before this commit: robot tmm_description, 12 links, 11 joints
Joints:
- joint SO101_joint1: limit lower=-2.0944 upper=2.0944 effort=10 velocity=10 -> lower=-2.0944 upper=2.0944 effort=1.9 velocity=4.4; origin xyz=-0.61481 -0.547483 0.11437 rpy=1.5708 -1.06378e-08 1.40416e-08 -> xyz=0.157389 0.000522483 -0.00526856 rpy=-3.14159 1.40141e-15 1.5708
- joint SO101_joint2: limit lower=-0.174533 upper=3.40339 effort=10 velocity=10 -> lower=-0.174533 upper=3.40339 effort=1.9 velocity=4.4
- joint SO101_joint3: limit lower=-3.31613 upper=0 effort=10 velocity=10 -> lower=-3.31613 upper=0 effort=1.9 velocity=4.4; origin xyz=0.11257 0.02795 -0.0007 rpy=9.96805e-17 1.15228e-14 -5.01053e-16 -> xyz=0.11257 0.02795 -0.0007 rpy=-6.08661e-18 -4.50966e-17 4.92007e-15
- joint SO101_joint4: limit lower=-1.74533 upper=1.74533 effort=10 velocity=10 -> lower=-1.74533 upper=1.74533 effort=1.9 velocity=4.4; origin xyz=-0.13485 0.00519806 -0.0007 rpy=-4.68315e-15 -5.23776e-17 1.5708 -> xyz=-0.13485 0.00519806 -0.0007 rpy=3.76281e-14 -5.94513e-17 1.5708
- joint SO101_joint5: limit lower=-2.87979 upper=2.87979 effort=10 velocity=10 -> lower=-2.87979 upper=2.87979 effort=1.9 velocity=4.4; type revolute -> continuous
- joint SO101_joint6: limit lower=-2.88658e-14 upper=2.26893 effort=10 velocity=10 -> lower=-0.174533 upper=2.0944 effort=1.9 velocity=4.4; origin xyz=0.0189497 -0.0198719 0.0233989 rpy=1.5708 -1.3963 1.58825 -> xyz=0.0189497 -0.0198719 0.0233989 rpy=-1.5708 -1.57076 -1.55334
- joint gimbal_joint1: origin xyz=-0.614052 -0.125414 -0.0274405 rpy=1.74311e-09 1.06378e-08 -3.14159 -> xyz=-0.0144218 0.00128011 0.4168 rpy=-1.5708 1.16573e-15 -1.5708
- joint gimbal_joint2: origin xyz=-0.01865 -0.0532 -0.01865 rpy=3.14159 1.5708 0 -> xyz=-0.01865 -0.0532 -0.01865 rpy=-3.14159 1.5708 0
- joint left_sprocket_joint: limit lower=-3.141592653589793 upper=3.141592653589793 effort=10 velocity=10 -> effort=10 velocity=10; origin xyz=-0.543758 -0.604353 -0.103839 rpy=1.5708 0.57871 -1.5708 -> xyz=-0.0608207 0.0715737 -0.0621391 rpy=1.5708 0.57871 -1.0148e-16; type revolute -> continuous
- joint right_sprocket_joint: limit lower=-3.141592653589793 upper=3.141592653589793 effort=10 velocity=10 -> effort=10 velocity=10; origin xyz=-0.68506 -0.604353 -0.103839 rpy=-1.5708 -0.57871 1.5708 -> xyz=-0.0608207 -0.0697275 -0.0621391 rpy=-1.5708 -0.57871 3.14159; type revolute -> continuous
